Commit message: fix(ares1): align STL origins to joint frames, remove head dome duplicate, visual/collision 0 0 0, limbs top-origin, Foxglove verified

File: src/ares1_description/urdf/ares1.urdf.xacro (robot description, xacro)
@@ -121,9 +121,9 @@
   <link name="neck_pitch_link"><inertial><mass value="4.0"/><inertia ixx="0.03" ixy="0" ixz="0" iyy="0.03" iyz="0" izz="0.02"/><origin xyz="0 0 0.06"/></inertial></link>
   <joint name="neck_pitch" type="revolute"><parent link="neck_base"/><child link="neck_pitch_link"/><origin xyz="0 0 0.08" rpy="0 0 0"/><axis xyz="0 1 0"/><limit lower="-0.524" upper="0.524" effort="120" velocity="2.0"/></joint>
-  <!-- ========== HEAD 280x260x240 + dome r90 12kg ========== -->
+  <!-- ========== HEAD 280x260x240 box ONLY 12kg (dome via sensor_dome) ========== -->
   <link name="head">
-    <inertial><mass value="${mass_head}"/><inertia ixx="0.18" ixy="0" ixz="0" iyy="0.16" iyz="0" izz="0.12"/><origin xyz="0 0 0.04"/></inertial>
-    <visual><geometry><mesh filename="package://ares1_description/meshes/visual/head.stl"/></geometry><material name="dark_grey"/></visual>
-    <collision><geometry><mesh filename="package://ares1_description/meshes/collision/head_col.stl"/></geometry></collision>
+    <inertial><mass value="${mass_head}"/><inertia ixx="0.18" ixy="0" ixz="0" iyy="0.16" iyz="0" izz="0.12"/><origin xyz="0 0 0.00"/></inertial>
+    <visual><origin xyz="0 0 0" rpy="0 0 0"/><geometry><mesh filename="package://ares1_description/meshes/visual/head.stl"/></geometry><material name="dark_grey"/></visual>
+    <collision><origin xyz="0 0 0" rpy="0 0 0"/><geometry><mesh filename="package://ares1_description/meshes/collision/head_col.stl"/></geometry></collision>
   </link>
   <joint name="head_joint" type="fixed"><parent link="neck_pitch_link"/><child link="head"/><origin xyz="0 0 0.07" rpy="0 0 0"/></joint>
@@ -173,9 +173,9 @@
       <axis xyz="0 1 0"/><limit lower="-3.14" upper="3.14" effort="280" velocity="2.5"/>
     </joint>
-    <!-- upper arm octagonal 380 -->
+    <!-- upper arm octagonal 380 — mesh origin at TOP (0 top, -0.38 bottom) -->
     <link name="${prefix}_upper_arm">
       <inertial><mass value="${mass_upper_arm}"/><inertia ixx="0.08" ixy="0" ixz="0" iyy="0.08" iyz="0" izz="0.04"/><origin xyz="0 0 -0.19"/></inertial>
-      <visual><origin xyz="0 0 -0.19" rpy="0 0 0"/><geometry><mesh filename="package://ares1_description/meshes/visual/upper_arm.stl"/></geometry><material name="dark_grey"/></visual>
-      <collision><geometry><mesh filename="package://ares1_description/meshes/collision/upper_arm_col.stl"/></geometry></collision>
+      <visual><origin xyz="0 0 0" rpy="0 0 0"/><geometry><mesh filename="package://ares1_description/meshes/visual/upper_arm.stl"/></geometry><material name="dark_grey"/></visual>
+      <collision><origin xyz="0 0 0" rpy="0 0 0"/><geometry><mesh filename="package://ares1_description/meshes/collision/upper_arm_col.stl"/></geometry></collision>
     </link>
     <joint name="${prefix}_upper_fixed" type="fixed"><parent link="${prefix}_shoulder_pitch"/><child link="${prefix}_upper_arm"/><origin xyz="0 0 -0.04" rpy="0 0 0"/></joint>
@@ -189,9 +189,9 @@
       <axis xyz="0 1 0"/><limit lower="0" upper="2.53" effort="200" velocity="2.5"/>
     </joint>
-    <!-- forearm 340 -->
+    <!-- forearm 340 — mesh origin at TOP -->
     <link name="${prefix}_forearm">
       <inertial><mass value="${mass_forearm}"/><inertia ixx="0.06" ixy="0" ixz="0" iyy="0.06" iyz="0" izz="0.03"/><origin xyz="0 0 -0.17"/></inertial>
-      <visual><origin xyz="0 0 -0.17" rpy="0 0 0"/><geometry><mesh filename="package://ares1_description/meshes/visual/forearm.stl"/></geometry><material name="dark_grey"/></visual>
-      <collision><geometry><mesh filename="package://ares1_description/meshes/collision/forearm_col.stl"/></geometry></collision>
+      <visual><origin xyz="0 0 0" rpy="0 0 0"/><geometry><mesh filename="package://ares1_description/meshes/visual/forearm.stl"/></geometry><material name="dark_grey"/></visual>
+      <collision><origin xyz="0 0 0" rpy="0 0 0"/><geometry><mesh filename="package://ares1_description/meshes/collision/forearm_col.stl"/></geometry></collision>
     </link>
     <joint name="${prefix}_forearm_fixed" type="fixed"><parent link="${prefix}_elbow_link"/><child link="${prefix}_forearm"/><origin xyz="0 0 0" rpy="0 0 0"/></joint>
@@ -222,6 +222,6 @@
     <link name="${prefix}_hand">
       <inertial><mass value="${mass_hand}"/><inertia ixx="0.02" ixy="0" ixz="0" iyy="0.02" iyz="0" izz="0.01"/><origin xyz="0 0 -0.08"/></inertial>
-      <visual><origin xyz="0 0 -0.08" rpy="0 0 0"/><geometry><mesh filename="package://ares1_description/meshes/visual/hand.stl"/></geometry><material name="gunmetal"/></visual>
-      <collision><geometry><mesh filename="package://ares1_description/meshes/collision/hand_col.stl"/></geometry></collision>
+      <visual><origin xyz="0 0 0" rpy="0 0 0"/><geometry><mesh filename="package://ares1_description/meshes/visual/hand.stl"/></geometry><material name="gunmetal"/></visual>
+      <collision><origin xyz="0 0 0" rpy="0 0 0"/><geometry><mesh filename="package://ares1_description/meshes/collision/hand_col.stl"/></geometry></collision>
     </link>
     <joint name="${prefix}_hand_joint" type="fixed"><parent link="${prefix}_wrist_roll"/><child link="${prefix}_hand"/><origin xyz="0 0 0" rpy="0 0 0"/></joint>
@@ -252,6 +252,6 @@
     <link name="${prefix}_thigh">
       <inertial><mass value="${mass_thigh}"/><inertia ixx="0.45" ixy="0" ixz="0" iyy="0.45" iyz="0" izz="0.12"/><origin xyz="0 0 -0.26"/></inertial>
-      <visual><origin xyz="0 0 -0.26" rpy="0 0 0"/><geometry><mesh filename="package://ares1_description/meshes/visual/thigh.stl"/></geometry><material name="dark_grey"/></visual>
-      <collision><geometry><mesh filename="package://ares1_description/meshes/collision/thigh_col.stl"/></geometry></collision>
+      <visual><origin xyz="0 0 0" rpy="0 0 0"/><geometry><mesh filename="package://ares1_description/meshes/visual/thigh.stl"/></geometry><material name="dark_grey"/></visual>
+      <collision><origin xyz="0 0 0" rpy="0 0 0"/><geometry><mesh filename="package://ares1_description/meshes/collision/thigh_col.stl"/></geometry></collision>
     </link>
     <joint name="${prefix}_thigh_joint" type="fixed"><parent link="${prefix}_hip_pitch"/><child link="${prefix}_thigh"/><origin xyz="0 0 0" rpy="0 0 0"/></joint>
@@ -260,6 +260,6 @@
     <link name="${prefix}_shin">
       <inertial><mass value="${mass_shin}"/><inertia ixx="0.28" ixy="0" ixz="0" iyy="0.28" iyz="0" izz="0.09"/><origin xyz="0 0 -0.24"/></inertial>
-      <visual><origin xyz="0 0 -0.24" rpy="0 0 0"/><geometry><mesh filename="package://ares1_description/meshes/visual/shin.stl"/></geometry><material name="dark_grey"/></visual>
-      <collision><geometry><mesh filename="package://ares1_description/meshes/collision/shin_col.stl"/></geometry></collision>
+      <visual><origin xyz="0 0 0" rpy="0 0 0"/><geometry><mesh filename="package://ares1_description/meshes/visual/shin.stl"/></geometry><material name="dark_grey"/></visual>
+      <collision><origin xyz="0 0 0" rpy="0 0 0"/><geometry><mesh filename="package://ares1_description/meshes/collision/shin_col.stl"/></geometry></collision>
     </link>
     <joint name="${prefix}_knee" type="revolute">
@@ -284,7 +284,7 @@
     </joint>
     <link name="${prefix}_foot">
-      <inertial><mass value="${mass_foot}"/><inertia ixx="0.04" ixy="0" ixz="0" iyy="0.06" iyz="0" izz="0.05"/><origin xyz="0.05 0 -0.02"/></inertial>
-      <visual><origin xyz="0.05 0 -0.02" rpy="0 0 0"/><geometry><mesh filename="package://ares1_description/meshes/visual/foot.stl"/></geometry><material name="gunmetal"/></visual>
-      <collision><geometry><mesh filename="package://ares1_description/meshes/collision/foot_col.stl"/></geometry></collision>
+      <inertial><mass value="${mass_foot}"/><inertia ixx="0.04" ixy="0" ixz="0" iyy="0.06" iyz="0" izz="0.05"/><origin xyz="0.00 0 -0.04"/></inertial>
+      <visual><origin xyz="0 0 0" rpy="0 0 0"/><geometry><mesh filename="package://ares1_description/meshes/visual/foot.stl"/></geometry><material name="gunmetal"/></visual>
+      <collision><origin xyz="0 0 0" rpy="0 0 0"/><geometry><mesh filename="package://ares1_description/meshes/collision/foot_col.stl"/></geometry></collision>
     </link>
     <joint name="${prefix}_foot_joint" type="fixed"><parent link="${prefix}_ankle_roll"/><child link="${prefix}_foot"/><origin xyz="0 0 0" rpy="0 0 0"/></joint>

Commit message: fix(ares1): aesthetic linked body — rpy align chest/pelvis/yoke to Y lateral, foot toe forward, joint ball housings, no floating plates

File: src/ares1_description/urdf/ares1.urdf.xacro (robot description, xacro)
@@ -28,5 +28,5 @@
   <material name="olive_drab"><color rgba="0.333 0.353 0.235 1.0"/></material>
   <material name="charcoal"><color rgba="0.216 0.216 0.227 1.0"/></material>
-  <!-- ========== PELVIS (base_link) — hex 460x260x180 22kg ========== -->
+  <!-- ========== PELVIS (base_link) — hex 460x260x180 22kg — rpy aligns width Y 460 depth X 260 -->
   <link name="base_link">
     <inertial>
@@ -36,9 +36,10 @@
     </inertial>
     <visual>
-      <origin xyz="0 0 0" rpy="0 0 0"/>
+      <origin xyz="0 0 0" rpy="0 0 1.5708"/>
       <geometry><mesh filename="package://ares1_description/meshes/visual/pelvis.stl" scale="1 1 1"/></geometry>
       <material name="dark_grey"/>
     </visual>
     <collision>
+      <origin xyz="0 0 0" rpy="0 0 1.5708"/>
       <geometry><mesh filename="package://ares1_description/meshes/collision/pelvis_col.stl" scale="1 1 1"/></geometry>
     </collision>
@@ -67,9 +68,9 @@
   </link>
   <joint name="abdomen3_fixed" type="fixed"><parent link="abdomen_ring2"/><child link="abdomen_ring3"/><origin xyz="0 0 0.085" rpy="0 0 0"/></joint>
-  <!-- ========== CHEST 520->440x280x380 32kg trapezoidal ========== -->
+  <!-- ========== CHEST 520->440x280x380 32kg trapezoidal — rpy aligns width Y 520 depth X 280 -->
   <link name="chest">
     <inertial><mass value="${mass_chest}"/><inertia ixx="1.2" ixy="0" ixz="0" iyy="1.0" iyz="0" izz="0.9"/><origin xyz="0 0 0"/></inertial>
-    <visual><geometry><mesh filename="package://ares1_description/meshes/visual/chest.stl"/></geometry><material name="dark_grey"/></visual>
-    <collision><geometry><mesh filename="package://ares1_description/meshes/collision/chest_col.stl"/></geometry></collision>
+    <visual><origin xyz="0 0 0" rpy="0 0 1.5708"/><geometry><mesh filename="package://ares1_description/meshes/visual/chest.stl"/></geometry><material name="dark_grey"/></visual>
+    <collision><origin xyz="0 0 0" rpy="0 0 1.5708"/><geometry><mesh filename="package://ares1_description/meshes/collision/chest_col.stl"/></geometry></collision>
   </link>
   <joint name="chest_joint" type="fixed"><parent link="abdomen_ring3"/><child link="chest"/><origin xyz="0 0 0.225" rpy="0 0 0"/></joint>
@@ -100,9 +101,9 @@
   <link name="fasteners"><inertial><mass value="4.8"/><inertia ixx="0.08" ixy="0" ixz="0" iyy="0.08" iyz="0" izz="0.06"/><origin xyz="0 0 0"/></inertial></link>
   <joint name="fasteners_joint" type="fixed"><parent link="base_link"/><child link="fasteners"/><origin xyz="0 0 0" rpy="0 0 0"/></joint>
-  <!-- ========== SHOULDER YOKE 640 span 80x120 14kg + pods ========== -->
+  <!-- ========== SHOULDER YOKE 640 span 80x120 14kg + pods — rpy aligns span Y 640 -->
   <link name="shoulder_yoke">
     <inertial><mass value="${mass_shoulder_yoke}"/><inertia ixx="0.45" ixy="0" ixz="0" iyy="0.85" iyz="0" izz="0.65"/><origin xyz="0 0 0"/></inertial>
-    <visual><geometry><mesh filename="package://ares1_description/meshes/visual/shoulder_yoke.stl"/></geometry><material name="gunmetal"/></visual>
-    <collision><geometry><mesh filename="package://ares1_description/meshes/collision/shoulder_yoke_col.stl"/></geometry></collision>
+    <visual><origin xyz="0 0 0" rpy="0 0 1.5708"/><geometry><mesh filename="package://ares1_description/meshes/visual/shoulder_yoke.stl"/></geometry><material name="gunmetal"/></visual>
+    <collision><origin xyz="0 0 0" rpy="0 0 1.5708"/><geometry><mesh filename="package://ares1_description/meshes/collision/shoulder_yoke_col.stl"/></geometry></collision>
   </link>
   <joint name="yoke_joint" type="fixed"><parent link="chest"/><child link="shoulder_yoke"/><origin xyz="0 0 0.235" rpy="0 0 0"/></joint>
@@ -154,6 +155,7 @@
   <!-- ========== ARMS 26-DOF detailed ========== -->
   <xacro:macro name="arm" params="prefix y">
-    <!-- shoulder 3 DOF: yaw->roll->pitch with dummy intermediates -->
-    <link name="${prefix}_shoulder_yaw"><inertial><mass value="0.5"/><inertia ixx="0.005" ixy="0" ixz="0" iyy="0.005" iyz="0" izz="0.005"/></inertial></link>
+    <!-- shoulder 3 DOF: yaw->roll->pitch — ball housing 110mm aesthetic -->
+    <link name="${prefix}_shoulder_yaw"><inertial><mass value="0.5"/><inertia ixx="0.005" ixy="0" ixz="0" iyy="0.005" iyz="0" izz="0.005"/></inertial>
+      <visual><origin xyz="0 0 0" rpy="0 0 0"/><geometry><sphere radius="0.055"/></geometry><material name="gunmetal"/></visual></link>
     <joint name="${prefix}_shoulder_yaw" type="revolute">
       <parent link="shoulder_yoke"/><child link="${prefix}_shoulder_yaw"/>
@@ -161,5 +163,6 @@
       <axis xyz="0 0 1"/><limit lower="-0.785" upper="0.785" effort="180" velocity="2.0"/>
     </joint>
-    <link name="${prefix}_shoulder_roll"><inertial><mass value="0.5"/><inertia ixx="0.005" ixy="0" ixz="0" iyy="0.005" iyz="0" izz="0.005"/></inertial></link>
+    <link name="${prefix}_shoulder_roll"><inertial><mass value="0.5"/><inertia ixx="0.005" ixy="0" ixz="0" iyy="0.005" iyz="0" izz="0.005"/></inertial>
+      <visual><origin xyz="0 0 0" rpy="0 0 0"/><geometry><sphere radius="0.050"/></geometry><material name="dark_grey"/></visual></link>
     <joint name="${prefix}_shoulder_roll" type="revolute">
       <parent link="${prefix}_shoulder_yaw"/><child link="${prefix}_shoulder_roll"/>
@@ -167,5 +170,6 @@
       <axis xyz="1 0 0"/><limit lower="-1.57" upper="1.57" effort="220" velocity="2.0"/>
     </joint>
-    <link name="${prefix}_shoulder_pitch"><inertial><mass value="1.0"/><inertia ixx="0.01" ixy="0" ixz="0" iyy="0.01" iyz="0" izz="0.01"/></inertial></link>
+    <link name="${prefix}_shoulder_pitch"><inertial><mass value="1.0"/><inertia ixx="0.01" ixy="0" ixz="0" iyy="0.01" iyz="0" izz="0.01"/></inertial>
+      <visual><origin xyz="0 0 0" rpy="0 0 0"/><geometry><sphere radius="0.045"/></geometry><material name="gunmetal"/></visual></link>
     <joint name="${prefix}_shoulder_pitch" type="revolute">
       <parent link="${prefix}_shoulder_roll"/><child link="${prefix}_shoulder_pitch"/>
@@ -180,8 +184,9 @@
     </link>
     <joint name="${prefix}_upper_fixed" type="fixed"><parent link="${prefix}_shoulder_pitch"/><child link="${prefix}_upper_arm"/><origin xyz="0 0 -0.04" rpy="0 0 0"/></joint>
-    <link name="armour_${prefix}_upper"><inertial><mass value="0.4"/><inertia ixx="0.005" ixy="0" ixz="0" iyy="0.005" iyz="0" izz="0.005"/></inertial><visual><origin xyz="0 0.02 -0.19" rpy="0 0 0"/><geometry><box size="0.008 0.04 0.20"/></geometry><material name="flat_black"/></visual></link>
+    <link name="armour_${prefix}_upper"><inertial><mass value="0.4"/><inertia ixx="0.005" ixy="0" ixz="0" iyy="0.005" iyz="0" izz="0.005"/></inertial><visual><origin xyz="0.064 0 -0.19" rpy="0 0 0"/><geometry><box size="0.012 0.04 0.20"/></geometry><material name="flat_black"/></visual></link>
     <joint name="armour_${prefix}_upper_joint" type="fixed"><parent link="${prefix}_upper_arm"/><child link="armour_${prefix}_upper"/><origin xyz="0 0 0" rpy="0 0 0"/></joint>
-    <!-- elbow -->
-    <link name="${prefix}_elbow_link"><inertial><mass value="0.3"/><inertia ixx="0.003" ixy="0" ixz="0" iyy="0.003" iyz="0" izz="0.002"/></inertial></link>
+    <!-- elbow — pin housing 85mm -->
+    <link name="${prefix}_elbow_link"><inertial><mass value="0.3"/><inertia ixx="0.003" ixy="0" ixz="0" iyy="0.003" iyz="0" izz="0.002"/></inertial>
+      <visual><origin xyz="0 0 0" rpy="0 1.5708 0"/><geometry><cylinder radius="0.042" length="0.10"/></geometry><material name="gunmetal"/></visual></link>
     <joint name="${prefix}_elbow" type="revolute">
       <parent link="${prefix}_upper_arm"/><child link="${prefix}_elbow_link"/>
@@ -196,5 +201,5 @@
     </link>
     <joint name="${prefix}_forearm_fixed" type="fixed"><parent link="${prefix}_elbow_link"/><child link="${prefix}_forearm"/><origin xyz="0 0 0" rpy="0 0 0"/></joint>
-    <link name="armour_${prefix}_forearm"><inertial><mass value="0.5"/><inertia ixx="0.006" ixy="0" ixz="0" iyy="0.006" iyz="0" izz="0.003"/></inertial><visual><origin xyz="0 0 -0.17" rpy="0 0 0"/><geometry><box size="0.012 0.06 0.20"/></geometry><material name="flat_black"/></visual></link>
+    <link name="armour_${prefix}_forearm"><inertial><mass value="0.5"/><inertia ixx="0.006" ixy="0" ixz="0" iyy="0.006" iyz="0" izz="0.003"/></inertial><visual><origin xyz="0.055 0 -0.17" rpy="0 0 0"/><geometry><box size="0.010 0.06 0.20"/></geometry><material name="flat_black"/></visual></link>
     <joint name="armour_${prefix}_forearm_joint" type="fixed"><parent link="${prefix}_forearm"/><child link="armour_${prefix}_forearm"/><origin xyz="0 0 0" rpy="0 0 0"/></joint>
     <!-- weapons per arm: left rifle SCAR-H 4.6kg 880mm, right grenade M320 1.5kg -->
@@ -207,6 +212,7 @@
       <joint name="${prefix}_launcher_joint" type="fixed"><parent link="${prefix}_forearm"/><child link="${prefix}_launcher"/><origin xyz="0.02 0 -0.34" rpy="0 0 0"/></joint>
     </xacro:if>
-    <!-- wrist 2 DOF -->
-    <link name="${prefix}_wrist_pitch"><inertial><mass value="0.6"/><inertia ixx="0.004" ixy="0" ixz="0" iyy="0.004" iyz="0" izz="0.002"/></inertial></link>
+    <!-- wrist 2 DOF — housing -->
+    <link name="${prefix}_wrist_pitch"><inertial><mass value="0.6"/><inertia ixx="0.004" ixy="0" ixz="0" iyy="0.004" iyz="0" izz="0.002"/></inertial>
+      <visual><origin xyz="0 0 0" rpy="0 0 0"/><geometry><cylinder radius="0.035" length="0.04"/></geometry><material name="dark_grey"/></visual></link>
     <joint name="${prefix}_wrist_pitch" type="revolute">
       <parent link="${prefix}_forearm"/><child link="${prefix}_wrist_pitch"/>
@@ -214,5 +220,6 @@
       <axis xyz="0 1 0"/><limit lower="-1.047" upper="1.047" effort="80" velocity="3.0"/>
     </joint>
-    <link name="${prefix}_wrist_roll"><inertial><mass value="0.5"/><inertia ixx="0.003" ixy="0" ixz="0" iyy="0.003" iyz="0" izz="0.002"/></inertial></link>
+    <link name="${prefix}_wrist_roll"><inertial><mass value="0.5"/><inertia ixx="0.003" ixy="0" ixz="0" iyy="0.003" iyz="0" izz="0.002"/></inertial>
+      <visual><origin xyz="0 0 0" rpy="0 0 0"/><geometry><sphere radius="0.030"/></geometry><material name="gunmetal"/></visual></link>
     <joint name="${prefix}_wrist_roll" type="revolute">
       <parent link="${prefix}_wrist_pitch"/><child link="${prefix}_wrist_roll"/>
@@ -231,6 +238,7 @@
   <!-- ========== LEGS 12 DOF (hip 3 + knee1 + ankle2 per leg) ========== -->
   <xacro:macro name="leg" params="prefix y">
-    <!-- hip yaw -> roll -> pitch dummy chain -->
-    <link name="${prefix}_hip_yaw"><inertial><mass value="0.8"/><inertia ixx="0.008" ixy="0" ixz="0" iyy="0.008" iyz="0" izz="0.008"/></inertial></link>
+    <!-- hip 3DOF — ball cup 95mm + hinge housings aesthetic -->
+    <link name="${prefix}_hip_yaw"><inertial><mass value="0.8"/><inertia ixx="0.008" ixy="0" ixz="0" iyy="0.008" iyz="0" izz="0.008"/></inertial>
+      <visual><origin xyz="0 0 0" rpy="0 0 0"/><geometry><sphere radius="0.050"/></geometry><material name="gunmetal"/></visual></link>
     <joint name="${prefix}_hip_yaw" type="revolute">
       <parent link="base_link"/><child link="${prefix}_hip_yaw"/>
@@ -238,5 +246,6 @@
       <axis xyz="0 0 1"/><limit lower="-0.524" upper="0.524" effort="200" velocity="2.0"/>
     </joint>
-    <link name="${prefix}_hip_roll"><inertial><mass value="0.8"/><inertia ixx="0.008" ixy="0" ixz="0" iyy="0.008" iyz="0" izz="0.008"/></inertial></link>
+    <link name="${prefix}_hip_roll"><inertial><mass value="0.8"/><inertia ixx="0.008" ixy="0" ixz="0" iyy="0.008" iyz="0" izz="0.008"/></inertial>
+      <visual><origin xyz="0 0 0" rpy="0 0 0"/><geometry><sphere radius="0.045"/></geometry><material name="dark_grey"/></visual></link>
     <joint name="${prefix}_hip_roll" type="revolute">
       <parent link="${prefix}_hip_yaw"/><child link="${prefix}_hip_roll"/>
@@ -244,5 +253,6 @@
       <axis xyz="1 0 0"/><limit lower="-0.785" upper="0.785" effort="280" velocity="2.0"/>
     </joint>
-    <link name="${prefix}_hip_pitch"><inertial><mass value="1.0"/><inertia ixx="0.01" ixy="0" ixz="0" iyy="0.01" iyz="0" izz="0.01"/></inertial></link>
+    <link name="${prefix}_hip_pitch"><inertial><mass value="1.0"/><inertia ixx="0.01" ixy="0" ixz="0" iyy="0.01" iyz="0" izz="0.01"/></inertial>
+      <visual><origin xyz="0 0 0" rpy="0 0 0"/><geometry><sphere radius="0.045"/></geometry><material name="gunmetal"/></visual></link>
     <joint name="${prefix}_hip_pitch" type="revolute">
       <parent link="${prefix}_hip_roll"/><child link="${prefix}_hip_pitch"/>
@@ -270,6 +280,7 @@
     <link name="armour_${prefix}_shin"><inertial><mass value="0.8"/><inertia ixx="0.015" ixy="0" ixz="0" iyy="0.015" iyz="0" izz="0.008"/><origin xyz="0 0 0"/></inertial><visual><origin xyz="0.07 0 -0.24" rpy="0 0 0"/><geometry><box size="0.015 0.10 0.28"/></geometry><material name="flat_black"/></visual></link>
     <joint name="armour_${prefix}_shin_joint" type="fixed"><parent link="${prefix}_shin"/><child link="armour_${prefix}_shin"/><origin xyz="0 0 0" rpy="0 0 0"/></joint>
-    <!-- ankle pitch -> roll -->
-    <link name="${prefix}_ankle_pitch"><inertial><mass value="0.6"/><inertia ixx="0.006" ixy="0" ixz="0" iyy="0.006" iyz="0" izz="0.004"/></inertial></link>
+    <!-- ankle pitch -> roll — gimbal housing 80mm -->
+    <link name="${prefix}_ankle_pitch"><inertial><mass value="0.6"/><inertia ixx="0.006" ixy="0" ixz="0" iyy="0.006" iyz="0" izz="0.004"/></inertial>
+      <visual><origin xyz="0 0 0" rpy="0 1.5708 0"/><geometry><cylinder radius="0.040" length="0.08"/></geometry><material name="dark_grey"/></visual></link>
     <joint name="${prefix}_ankle_pitch" type="revolute">
       <parent link="${prefix}_shin"/><child link="${prefix}_ankle_pitch"/>
@@ -277,5 +288,6 @@
       <axis xyz="0 1 0"/><limit lower="-0.698" upper="0.698" effort="220" velocity="3.0"/>
     </joint>
-    <link name="${prefix}_ankle_roll"><inertial><mass value="0.5"/><inertia ixx="0.005" ixy="0" ixz="0" iyy="0.005" iyz="0" izz="0.003"/></inertial></link>
+    <link name="${prefix}_ankle_roll"><inertial><mass value="0.5"/><inertia ixx="0.005" ixy="0" ixz="0" iyy="0.005" iyz="0" izz="0.003"/></inertial>
+      <visual><origin xyz="0 0 0" rpy="0 0 0"/><geometry><sphere radius="0.035"/></geometry><material name="gunmetal"/></visual></link>
     <joint name="${prefix}_ankle_roll" type="revolute">
       <parent link="${prefix}_ankle_pitch"/><child link="${prefix}_ankle_roll"/>
