Commit message: clean(ares1): weapon-free no mounts 402kg 62/61 (was 69/68) — remove shield/pods/drones/rifle/launcher, chest 39.75kg, controllers 26-DOF only, cors http 8000, delete single_color 24M

File: src/ares1_description/urdf/ares1.urdf.xacro (robot description, xacro)
@@ -1,11 +1,11 @@
 <?xml version="1.0"?>
 <robot xmlns:xacro="http://www.ros.org/wiki/xacro" name="ares1">
-  <!-- ARES-1 v1.0 arc.md complete spec — 2430mm 447kg 26-DOF mesh STL -->
+  <!-- ARES-1 v1.0 weapon-free 402kg 26-DOF — mounts removed per user, high 50K 46K faces -->
   <!-- Meshes generated procedural at src/ares1_description/meshes/visual/*.stl scale 1 (meters) -->
-  <!-- Height stack arc.md: foot80 + shin480 + knee60 + thigh520 + hip60 + pelvis180 + abdomen220 + chest380 + neck120 + head240 + dome90 = 2430 -->
-  <!-- Weight budget arc.md: 447kg detailed -->
+  <!-- Height stack: foot80 + shin480 + knee60 + thigh520 + hip60 + pelvis180 + abdomen220 + chest380 + neck120 + head240 + dome90 = 2430 -->
+  <!-- Weight budget: 402kg weapon-free (447kg - shield18 - pods26.4 - drones2.25 - rifle4.6 - launcher1.5 =394.3 +7.7 redistributed to chest) -->
   <xacro:property name="mass_head" value="12.0"/>
   <xacro:property name="mass_neck" value="6.0"/>
-  <xacro:property name="mass_chest" value="32.0"/>
+  <xacro:property name="mass_chest" value="39.75"/>
   <xacro:property name="mass_abdomen_ring" value="4.0"/>
   <xacro:property name="mass_pelvis" value="22.0"/>
@@ -108,9 +108,5 @@
   </link>
   <joint name="yoke_joint" type="fixed"><parent link="chest"/><child link="shoulder_yoke"/><origin xyz="0 0 0.235" rpy="0 0 0"/></joint>
-  <!-- Missile pods 400x80x80 each 1.2kg + 3 missiles 4kg each -->
-  <link name="pod_left"><inertial><mass value="13.2"/><inertia ixx="0.18" ixy="0" ixz="0" iyy="0.18" iyz="0" izz="0.06"/><origin xyz="0 0 0"/></inertial><visual><geometry><mesh filename="package://ares1_description/meshes/visual/missile_pod.stl"/></geometry><material name="olive_drab"/></visual><collision><geometry><mesh filename="package://ares1_description/meshes/collision/missile_pod_col.stl"/></geometry></collision></link>
-  <joint name="pod_left_joint" type="revolute"><parent link="shoulder_yoke"/><child link="pod_left"/><origin xyz="0 0.28 0.06" rpy="0 0 0"/><axis xyz="0 1 0"/><limit lower="0" upper="0.785" effort="30" velocity="1.0"/></joint>
-  <link name="pod_right"><inertial><mass value="13.2"/><inertia ixx="0.18" ixy="0" ixz="0" iyy="0.18" iyz="0" izz="0.06"/><origin xyz="0 0 0"/></inertial><visual><geometry><mesh filename="package://ares1_description/meshes/visual/missile_pod.stl"/></geometry><material name="olive_drab"/></visual><collision><geometry><mesh filename="package://ares1_description/meshes/collision/missile_pod_col.stl"/></geometry></collision></link>
-  <joint name="pod_right_joint" type="revolute"><parent link="shoulder_yoke"/><child link="pod_right"/><origin xyz="0 -0.28 0.06" rpy="0 0 0"/><axis xyz="0 1 0"/><limit lower="0" upper="0.785" effort="30" velocity="1.0"/></joint>
+  <!-- Missile pods removed — weapon-free clean no mounts (re-add after build) -->
   <!-- ========== NECK 70->90x120 6kg 2-DOF ========== -->
   <link name="neck_base">
@@ -135,22 +131,5 @@
   <link name="sensor_dome"><inertial><mass value="0.5"/><inertia ixx="0.005" ixy="0" ixz="0" iyy="0.005" iyz="0" izz="0.005"/></inertial><visual><origin xyz="0 0 0.14" rpy="0 0 0"/><geometry><sphere radius="0.09"/></geometry><material name="visor_blue"/></visual></link>
   <joint name="dome_joint" type="fixed"><parent link="head"/><child link="sensor_dome"/><origin xyz="0 0 0" rpy="0 0 0"/></joint>
-  <!-- ========== DRONE BAYS (left fixed 1.4kg, right quad 0.85kg) per arc.md 459 ========== -->
-  <link name="drone_fixed_wing"><inertial><mass value="${mass_drone_fixed}"/><inertia ixx="0.02" ixy="0" ixz="0" iyy="0.02" iyz="0" izz="0.015"/><origin xyz="0 0 0"/></inertial><visual><geometry><mesh filename="package://ares1_description/meshes/visual/drone_fixed_wing.stl"/></geometry><material name="flat_black"/></visual></link>
-  <joint name="drone1_fixed" type="fixed"><parent link="chest"/><child link="drone_fixed_wing"/><origin xyz="-0.16 0.11 -0.08" rpy="0 0 0"/></joint>
-  <link name="drone_quad"><inertial><mass value="${mass_drone_quad}"/><inertia ixx="0.01" ixy="0" ixz="0" iyy="0.01" iyz="0" izz="0.008"/><origin xyz="0 0 0"/></inertial><visual><geometry><mesh filename="package://ares1_description/meshes/visual/drone_quad.stl"/></geometry><material name="flat_black"/></visual></link>
-  <joint name="drone2_fixed" type="fixed"><parent link="chest"/><child link="drone_quad"/><origin xyz="-0.16 -0.11 -0.08" rpy="0 0 0"/></joint>
-  <!-- ========== SHIELD 1200x700x48 18kg B4C+UHMWPE+Ti ========== -->
-  <link name="shield">
-    <inertial><mass value="${mass_shield}"/><inertia ixx="2.1" ixy="0" ixz="0" iyy="0.9" iyz="0" izz="2.4"/><origin xyz="0 0 0.60"/></inertial>
-    <visual><geometry><mesh filename="package://ares1_description/meshes/visual/shield.stl"/></geometry><material name="charcoal"/></visual>
-    <collision><geometry><mesh filename="package://ares1_description/meshes/collision/shield_col.stl"/></geometry></collision>
-  </link>
-  <joint name="shield_pivot" type="revolute">
-    <parent link="shoulder_yoke"/><child link="shield"/>
-    <origin xyz="0 0.32 0.0" rpy="0 0 0"/>
-    <axis xyz="0 1 0"/>
-    <limit lower="0" upper="1.83" effort="500" velocity="3.5"/>
-    <dynamics damping="12" friction="3"/>
-  </joint>
+  <!-- Drone bays & shield removed — weapon-free clean no mounts (re-add after build) -->
   <!-- ========== ARMS 26-DOF detailed ========== -->
   <xacro:macro name="arm" params="prefix y">
@@ -203,13 +182,5 @@
     <link name="armour_${prefix}_forearm"><inertial><mass value="0.5"/><inertia ixx="0.006" ixy="0" ixz="0" iyy="0.006" iyz="0" izz="0.003"/></inertial><visual><origin xyz="0.055 0 -0.17" rpy="0 0 0"/><geometry><box size="0.010 0.06 0.20"/></geometry><material name="flat_black"/></visual></link>
     <joint name="armour_${prefix}_forearm_joint" type="fixed"><parent link="${prefix}_forearm"/><child link="armour_${prefix}_forearm"/><origin xyz="0 0 0" rpy="0 0 0"/></joint>
-    <!-- weapons per arm: left rifle SCAR-H 4.6kg 880mm, right grenade M320 1.5kg -->
-    <xacro:if value="${prefix == 'left'}">
-      <link name="${prefix}_rifle"><inertial><mass value="4.6"/><inertia ixx="0.05" ixy="0" ixz="0" iyy="0.05" iyz="0" izz="0.02"/><origin xyz="0.44 0 0"/></inertial><visual><origin xyz="0.44 0 0" rpy="0 1.57 0"/><geometry><box size="0.88 0.04 0.06"/></geometry><material name="olive_drab"/></visual></link>
-      <joint name="${prefix}_rifle_joint" type="fixed"><parent link="${prefix}_forearm"/><child link="${prefix}_rifle"/><origin xyz="0 0 -0.34" rpy="0 0 0"/></joint>
-    </xacro:if>
-    <xacro:if value="${prefix == 'right'}">
-      <link name="${prefix}_launcher"><inertial><mass value="1.5"/><inertia ixx="0.01" ixy="0" ixz="0" iyy="0.01" iyz="0" izz="0.005"/><origin xyz="0 0 -0.12"/></inertial><visual><origin xyz="0 0 -0.12" rpy="0 1.57 0"/><geometry><box size="0.23 0.04 0.04"/></geometry><material name="olive_drab"/></visual></link>
-      <joint name="${prefix}_launcher_joint" type="fixed"><parent link="${prefix}_forearm"/><child link="${prefix}_launcher"/><origin xyz="0.02 0 -0.34" rpy="0 0 0"/></joint>
-    </xacro:if>
+    <!-- weapons removed — clean no mounts -->
     <!-- wrist 2 DOF — housing -->
     <link name="${prefix}_wrist_pitch"><inertial><mass value="0.6"/><inertia ixx="0.004" ixy="0" ixz="0" iyy="0.004" iyz="0" izz="0.002"/></inertial>
@@ -344,4 +315,3 @@
     <sensor name="right_ft" type="force_torque"><always_on>true</always_on><update_rate>1000</update_rate><topic>/ares1/sensors/foot/right/ft</topic></sensor>
   </gazebo>
-  <gazebo reference="shield"><material>Gazebo/Charcoal</material></gazebo>
 </robot>

Commit message: feat(ares1): Option B detailed 159 loose parts from Drive FBX — delete old 16 high50K entirely, 159 part_*.stl 41K faces 62 links 61 joints 402kg, detailed_visuals.xacro base_link 159 visuals, weapon-free clean no mounts

File: src/ares1_description/urdf/ares1.urdf.xacro (robot description, xacro)
@@ -1,4 +1,5 @@
 <?xml version="1.0"?>
 <robot xmlns:xacro="http://www.ros.org/wiki/xacro" name="ares1">
+  <xacro:include filename="$(find ares1_description)/urdf/detailed_visuals.xacro"/>
   <!-- ARES-1 v1.0 weapon-free 402kg 26-DOF — mounts removed per user, high 50K 46K faces -->
   <!-- Meshes generated procedural at src/ares1_description/meshes/visual/*.stl scale 1 (meters) -->
@@ -37,10 +38,11 @@
     <visual>
       <origin xyz="0 0 0" rpy="0 0 1.5708"/>
-      <geometry><mesh filename="package://ares1_description/meshes/visual/pelvis.stl" scale="1 1 1"/></geometry>
+      <geometry><box size="0.46 0.26 0.18"/></geometry>
       <material name="dark_grey"/>
     </visual>
+    <xacro:detailed_visuals/>
     <collision>
       <origin xyz="0 0 0" rpy="0 0 1.5708"/>
-      <geometry><mesh filename="package://ares1_description/meshes/collision/pelvis_col.stl" scale="1 1 1"/></geometry>
+      <geometry><box size="0.46 0.26 0.18"/></geometry>
     </collision>
   </link>
@@ -52,18 +54,18 @@
   <link name="abdomen_ring1">
     <inertial><mass value="${mass_abdomen_ring}"/><inertia ixx="0.12" ixy="0" ixz="0" iyy="0.12" iyz="0" izz="0.08"/><origin xyz="0 0 0"/></inertial>
-    <visual><geometry><mesh filename="package://ares1_description/meshes/visual/abdomen_ring.stl" scale="1 1 1"/></geometry><material name="dark_grey"/></visual>
-    <collision><geometry><mesh filename="package://ares1_description/meshes/collision/abdomen_ring_col.stl"/></geometry></collision>
+    <visual><geometry><cylinder radius="0.18" length="0.06"/></geometry><material name="dark_grey"/></visual>
+    <collision><geometry><cylinder radius="0.18" length="0.06"/></geometry></collision>
   </link>
   <joint name="abdomen1_fixed" type="fixed"><parent link="base_link"/><child link="abdomen_ring1"/><origin xyz="0 0 0.115" rpy="0 0 0"/></joint>
   <link name="abdomen_ring2">
     <inertial><mass value="${mass_abdomen_ring}"/><inertia ixx="0.12" ixy="0" ixz="0" iyy="0.12" iyz="0" izz="0.08"/><origin xyz="0 0 0"/></inertial>
-    <visual><geometry><mesh filename="package://ares1_description/meshes/visual/abdomen_ring.stl"/></geometry><material name="flat_black"/></visual>
-    <collision><geometry><mesh filename="package://ares1_description/meshes/collision/abdomen_ring_col.stl"/></geometry></collision>
+    <visual><geometry><cylinder radius="0.18" length="0.06"/></geometry><material name="flat_black"/></visual>
+    <collision><geometry><cylinder radius="0.18" length="0.06"/></geometry></collision>
   </link>
   <joint name="abdomen2_fixed" type="fixed"><parent link="abdomen_ring1"/><child link="abdomen_ring2"/><origin xyz="0 0 0.085" rpy="0 0 0"/></joint>
   <link name="abdomen_ring3">
     <inertial><mass value="${mass_abdomen_ring}"/><inertia ixx="0.12" ixy="0" ixz="0" iyy="0.12" iyz="0" izz="0.08"/><origin xyz="0 0 0"/></inertial>
-    <visual><geometry><mesh filename="package://ares1_description/meshes/visual/abdomen_ring.stl"/></geometry><material name="dark_grey"/></visual>
-    <collision><geometry><mesh filename="package://ares1_description/meshes/collision/abdomen_ring_col.stl"/></geometry></collision>
+    <visual><geometry><cylinder radius="0.18" length="0.06"/></geometry><material name="dark_grey"/></visual>
+    <collision><geometry><cylinder radius="0.18" length="0.06"/></geometry></collision>
   </link>
   <joint name="abdomen3_fixed" type="fixed"><parent link="abdomen_ring2"/><child link="abdomen_ring3"/><origin xyz="0 0 0.085" rpy="0 0 0"/></joint>
@@ -71,6 +73,6 @@
   <link name="chest">
     <inertial><mass value="${mass_chest}"/><inertia ixx="1.2" ixy="0" ixz="0" iyy="1.0" iyz="0" izz="0.9"/><origin xyz="0 0 0"/></inertial>
-    <visual><origin xyz="0 0 0" rpy="0 0 1.5708"/><geometry><mesh filename="package://ares1_description/meshes/visual/chest.stl"/></geometry><material name="dark_grey"/></visual>
-    <collision><origin xyz="0 0 0" rpy="0 0 1.5708"/><geometry><mesh filename="package://ares1_description/meshes/collision/chest_col.stl"/></geometry></collision>
+    <visual><origin xyz="0 0 0" rpy="0 0 1.5708"/><geometry><box size="0.28 0.52 0.38"/></geometry><material name="dark_grey"/></visual>
+    <collision><origin xyz="0 0 0" rpy="0 0 1.5708"/><geometry><box size="0.28 0.52 0.38"/></geometry></collision>
   </link>
   <joint name="chest_joint" type="fixed"><parent link="abdomen_ring3"/><child link="chest"/><origin xyz="0 0 0.225" rpy="0 0 0"/></joint>
@@ -104,6 +106,6 @@
   <link name="shoulder_yoke">
     <inertial><mass value="${mass_shoulder_yoke}"/><inertia ixx="0.45" ixy="0" ixz="0" iyy="0.85" iyz="0" izz="0.65"/><origin xyz="0 0 0"/></inertial>
-    <visual><origin xyz="0 0 0" rpy="0 0 1.5708"/><geometry><mesh filename="package://ares1_description/meshes/visual/shoulder_yoke.stl"/></geometry><material name="gunmetal"/></visual>
-    <collision><origin xyz="0 0 0" rpy="0 0 1.5708"/><geometry><mesh filename="package://ares1_description/meshes/collision/shoulder_yoke_col.stl"/></geometry></collision>
+    <visual><origin xyz="0 0 0" rpy="0 0 1.5708"/><geometry><box size="0.12 0.64 0.08"/></geometry><material name="gunmetal"/></visual>
+    <collision><origin xyz="0 0 0" rpy="0 0 1.5708"/><geometry><box size="0.12 0.64 0.08"/></geometry></collision>
   </link>
   <joint name="yoke_joint" type="fixed"><parent link="chest"/><child link="shoulder_yoke"/><origin xyz="0 0 0.235" rpy="0 0 0"/></joint>
@@ -112,6 +114,6 @@
   <link name="neck_base">
     <inertial><mass value="2.0"/><inertia ixx="0.02" ixy="0" ixz="0" iyy="0.02" iyz="0" izz="0.01"/><origin xyz="0 0 0"/></inertial>
-    <visual><geometry><mesh filename="package://ares1_description/meshes/visual/neck.stl"/></geometry><material name="gunmetal"/></visual>
-    <collision><geometry><mesh filename="package://ares1_description/meshes/collision/neck_col.stl"/></geometry></collision>
+    <visual><geometry><cylinder radius="0.045" length="0.12"/></geometry><material name="gunmetal"/></visual>
+    <collision><geometry><cylinder radius="0.045" length="0.12"/></geometry></collision>
   </link>
   <joint name="neck_yaw" type="revolute"><parent link="chest"/><child link="neck_base"/><origin xyz="0 0 0.250" rpy="0 0 0"/><axis xyz="0 0 1"/><limit lower="-1.57" upper="1.57" effort="120" velocity="2.0"/><dynamics damping="5" friction="1"/></joint>
@@ -121,6 +123,6 @@
   <link name="head">
     <inertial><mass value="${mass_head}"/><inertia ixx="0.18" ixy="0" ixz="0" iyy="0.16" iyz="0" izz="0.12"/><origin xyz="0 0 0.00"/></inertial>
-    <visual><origin xyz="0 0 0" rpy="0 0 0"/><geometry><mesh filename="package://ares1_description/meshes/visual/head.stl"/></geometry><material name="dark_grey"/></visual>
-    <collision><origin xyz="0 0 0" rpy="0 0 0"/><geometry><mesh filename="package://ares1_description/meshes/collision/head_col.stl"/></geometry></collision>
+    <visual><origin xyz="0 0 0" rpy="0 0 0"/><geometry><box size="0.28 0.26 0.24"/></geometry><material name="dark_grey"/></visual>
+    <collision><origin xyz="0 0 0" rpy="0 0 0"/><geometry><box size="0.28 0.26 0.24"/></geometry></collision>
   </link>
   <joint name="head_joint" type="fixed"><parent link="neck_pitch_link"/><child link="head"/><origin xyz="0 0 0.07" rpy="0 0 0"/></joint>
@@ -159,6 +161,6 @@
     <link name="${prefix}_upper_arm">
       <inertial><mass value="${mass_upper_arm}"/><inertia ixx="0.08" ixy="0" ixz="0" iyy="0.08" iyz="0" izz="0.04"/><origin xyz="0 0 -0.19"/></inertial>
-      <visual><origin xyz="0 0 0" rpy="0 0 0"/><geometry><mesh filename="package://ares1_description/meshes/visual/upper_arm.stl"/></geometry><material name="dark_grey"/></visual>
-      <collision><origin xyz="0 0 0" rpy="0 0 0"/><geometry><mesh filename="package://ares1_description/meshes/collision/upper_arm_col.stl"/></geometry></collision>
+      <visual><origin xyz="0 0 0" rpy="0 0 0"/><geometry><cylinder radius="0.055" length="0.38"/></geometry><material name="dark_grey"/></visual>
+      <collision><origin xyz="0 0 0" rpy="0 0 0"/><geometry><cylinder radius="0.055" length="0.38"/></geometry></collision>
     </link>
     <joint name="${prefix}_upper_fixed" type="fixed"><parent link="${prefix}_shoulder_pitch"/><child link="${prefix}_upper_arm"/><origin xyz="0 0 -0.04" rpy="0 0 0"/></joint>
@@ -176,6 +178,6 @@
     <link name="${prefix}_forearm">
       <inertial><mass value="${mass_forearm}"/><inertia ixx="0.06" ixy="0" ixz="0" iyy="0.06" iyz="0" izz="0.03"/><origin xyz="0 0 -0.17"/></inertial>
-      <visual><origin xyz="0 0 0" rpy="0 0 0"/><geometry><mesh filename="package://ares1_description/meshes/visual/forearm.stl"/></geometry><material name="dark_grey"/></visual>
-      <collision><origin xyz="0 0 0" rpy="0 0 0"/><geometry><mesh filename="package://ares1_description/meshes/collision/forearm_col.stl"/></geometry></collision>
+      <visual><origin xyz="0 0 0" rpy="0 0 0"/><geometry><cylinder radius="0.045" length="0.34"/></geometry><material name="dark_grey"/></visual>
+      <collision><origin xyz="0 0 0" rpy="0 0 0"/><geometry><cylinder radius="0.045" length="0.34"/></geometry></collision>
     </link>
     <joint name="${prefix}_forearm_fixed" type="fixed"><parent link="${prefix}_elbow_link"/><child link="${prefix}_forearm"/><origin xyz="0 0 0" rpy="0 0 0"/></joint>
@@ -200,6 +202,6 @@
     <link name="${prefix}_hand">
       <inertial><mass value="${mass_hand}"/><inertia ixx="0.02" ixy="0" ixz="0" iyy="0.02" iyz="0" izz="0.01"/><origin xyz="0 0 -0.08"/></inertial>
-      <visual><origin xyz="0 0 0" rpy="0 0 0"/><geometry><mesh filename="package://ares1_description/meshes/visual/hand.stl"/></geometry><material name="gunmetal"/></visual>
-      <collision><origin xyz="0 0 0" rpy="0 0 0"/><geometry><mesh filename="package://ares1_description/meshes/collision/hand_col.stl"/></geometry></collision>
+      <visual><origin xyz="0 0 0" rpy="0 0 0"/><geometry><box size="0.095 0.085 0.11"/></geometry><material name="gunmetal"/></visual>
+      <collision><origin xyz="0 0 0" rpy="0 0 0"/><geometry><box size="0.095 0.085 0.11"/></geometry></collision>
     </link>
     <joint name="${prefix}_hand_joint" type="fixed"><parent link="${prefix}_wrist_roll"/><child link="${prefix}_hand"/><origin xyz="0 0 0" rpy="0 0 0"/></joint>
@@ -233,6 +235,6 @@
     <link name="${prefix}_thigh">
       <inertial><mass value="${mass_thigh}"/><inertia ixx="0.45" ixy="0" ixz="0" iyy="0.45" iyz="0" izz="0.12"/><origin xyz="0 0 -0.26"/></inertial>
-      <visual><origin xyz="0 0 0" rpy="0 0 0"/><geometry><mesh filename="package://ares1_description/meshes/visual/thigh.stl"/></geometry><material name="dark_grey"/></visual>
-      <collision><origin xyz="0 0 0" rpy="0 0 0"/><geometry><mesh filename="package://ares1_description/meshes/collision/thigh_col.stl"/></geometry></collision>
+      <visual><origin xyz="0 0 0" rpy="0 0 0"/><geometry><cylinder radius="0.10" length="0.52"/></geometry><material name="dark_grey"/></visual>
+      <collision><origin xyz="0 0 0" rpy="0 0 0"/><geometry><cylinder radius="0.10" length="0.52"/></geometry></collision>
     </link>
     <joint name="${prefix}_thigh_joint" type="fixed"><parent link="${prefix}_hip_pitch"/><child link="${prefix}_thigh"/><origin xyz="0 0 0" rpy="0 0 0"/></joint>
@@ -241,6 +243,6 @@
     <link name="${prefix}_shin">
       <inertial><mass value="${mass_shin}"/><inertia ixx="0.28" ixy="0" ixz="0" iyy="0.28" iyz="0" izz="0.09"/><origin xyz="0 0 -0.24"/></inertial>
-      <visual><origin xyz="0 0 0" rpy="0 0 0"/><geometry><mesh filename="package://ares1_description/meshes/visual/shin.stl"/></geometry><material name="dark_grey"/></visual>
-      <collision><origin xyz="0 0 0" rpy="0 0 0"/><geometry><mesh filename="package://ares1_description/meshes/collision/shin_col.stl"/></geometry></collision>
+      <visual><origin xyz="0 0 0" rpy="0 0 0"/><geometry><cylinder radius="0.08" length="0.48"/></geometry><material name="dark_grey"/></visual>
+      <collision><origin xyz="0 0 0" rpy="0 0 0"/><geometry><cylinder radius="0.08" length="0.48"/></geometry></collision>
     </link>
     <joint name="${prefix}_knee" type="revolute">
@@ -268,6 +270,6 @@
     <link name="${prefix}_foot">
       <inertial><mass value="${mass_foot}"/><inertia ixx="0.04" ixy="0" ixz="0" iyy="0.06" iyz="0" izz="0.05"/><origin xyz="0.00 0 -0.04"/></inertial>
-      <visual><origin xyz="0 0 0" rpy="0 0 0"/><geometry><mesh filename="package://ares1_description/meshes/visual/foot.stl"/></geometry><material name="gunmetal"/></visual>
-      <collision><origin xyz="0 0 0" rpy="0 0 0"/><geometry><mesh filename="package://ares1_description/meshes/collision/foot_col.stl"/></geometry></collision>
+      <visual><origin xyz="0 0 0" rpy="0 0 0"/><geometry><box size="0.24 0.20 0.045"/></geometry><material name="gunmetal"/></visual>
+      <collision><origin xyz="0 0 0" rpy="0 0 0"/><geometry><box size="0.24 0.20 0.045"/></geometry></collision>
     </link>
     <joint name="${prefix}_foot_joint" type="fixed"><parent link="${prefix}_ankle_roll"/><child link="${prefix}_foot"/><origin xyz="0 0 0" rpy="0 0 0"/></joint>
