Commit message: fix(ares1): upright humanoid - continuous torso, Y->Z half-length offsets, recenter hip/palm
- torso continuous: pelvis(0.283)->abdominal(0.266)->chest(0.356)->neck(0.166)->head(0.224)
  joints abdomen1 0.274, abdomen2/3 0.266, chest 0.311, neck 0.261 based on trimesh half-sizes
- arms/legs Y-axis meshes rpy 1.5708 0 0 with -half Z: upper_arm -0.1715, forearm -0.129, thigh -0.25, calf -0.2255, palm -0.082
- foot Z-long 0.299 -> rpy 1.5708 0 1.5708 xyz 0.10 0 -0.0925 (forward X)
- recenter hip_joint/palm STL/OBJ from world-offset to link-local
- regenerate ares1.urdf, remove box/cylinder/sphere primitives (21 mesh visuals remain)
- foxglove asset allowlist .* for package:// loading

File: ares1.urdf (robot description, URDF)
Before this commit: robot ares1, 69 links, 68 joints
Links:
- removed link drone_fixed_wing
- removed link drone_quad
- removed link left_rifle
- removed link pod_left
- removed link pod_right
- removed link right_launcher
- removed link shield
- link abdomen_ring1: geometry collision mesh filename=package://ares1_description/meshes/collision/abdominal.obj; visual mesh filename=package://ares1_description/meshes/visual/abdominal.obj scale=1 1 1
- link abdomen_ring2: geometry collision mesh filename=package://ares1_description/meshes/collision/abdominal.obj; visual mesh filename=package://ares1_description/meshes/visual/abdominal.obj scale=1 1 1
- link abdomen_ring3: geometry collision mesh filename=package://ares1_description/meshes/collision/abdominal.obj; visual mesh filename=package://ares1_description/meshes/visual/abdominal.obj
- link armour_back: geometry 
- link armour_chest_front: geometry 
- link armour_head_front: geometry 
- link armour_left_forearm: geometry 
- link armour_left_shin: geometry 
- link armour_left_thigh: geometry 
- link armour_left_upper: geometry 
- link armour_right_forearm: geometry 
- link armour_right_shin: geometry 
- link armour_right_thigh: geometry 
- link armour_right_upper: geometry 
- link base_link: geometry collision mesh filename=package://ares1_description/meshes/collision/pelvis.obj scale=1 1 1; visual mesh filename=package://ares1_description/meshes/visual/pelvis.obj scale=1 1 1
- link chest: mass 32.0 -> 39.75; geometry collision mesh filename=package://ares1_description/meshes/collision/chest.obj; visual mesh filename=package://ares1_description/meshes/visual/chest.obj scale=1 1 1
- link head: geometry collision mesh filename=package://ares1_description/meshes/collision/head.obj; visual mesh filename=package://ares1_description/meshes/visual/head.obj scale=1 1 1
- link left_foot: geometry collision mesh filename=package://ares1_description/meshes/collision/foot_L.obj; visual mesh filename=package://ares1_description/meshes/visual/foot_L.obj
- link left_forearm: geometry collision mesh filename=package://ares1_description/meshes/collision/forearm_L.obj; visual mesh filename=package://ares1_description/meshes/visual/forearm_L.obj
- link left_hand: geometry collision mesh filename=package://ares1_description/meshes/collision/palm_L.obj; visual mesh filename=package://ares1_description/meshes/visual/palm_L.obj
- link left_hip_yaw: geometry visual mesh filename=package://ares1_description/meshes/visual/hip_joint_L.obj scale=1 1 1
- link left_shin: geometry collision mesh filename=package://ares1_description/meshes/collision/calf_L.obj; visual mesh filename=package://ares1_description/meshes/visual/calf_L.obj
- link left_thigh: geometry collision mesh filename=package://ares1_description/meshes/collision/thigh_L.obj; visual mesh filename=package://ares1_description/meshes/visual/thigh_L.obj
- link left_upper_arm: geometry collision mesh filename=package://ares1_description/meshes/collision/upper_arm_L.obj; visual mesh filename=package://ares1_description/meshes/visual/upper_arm_L.obj
- link neck_base: geometry collision mesh filename=package://ares1_description/meshes/collision/neck.obj; visual mesh filename=package://ares1_description/meshes/visual/neck.obj scale=1 1 1
- link right_foot: geometry collision mesh filename=package://ares1_description/meshes/collision/foot_R.obj; visual mesh filename=package://ares1_description/meshes/visual/foot_R.obj
- link right_forearm: geometry collision mesh filename=package://ares1_description/meshes/collision/forearm_R.obj; visual mesh filename=package://ares1_description/meshes/visual/forearm_R.obj
- link right_hand: geometry collision mesh filename=package://ares1_description/meshes/collision/palm_R.obj; visual mesh filename=package://ares1_description/meshes/visual/palm_R.obj
- link right_hip_yaw: geometry visual mesh filename=package://ares1_description/meshes/visual/hip_joint_R.obj scale=1 1 1
- link right_shin: geometry collision mesh filename=package://ares1_description/meshes/collision/calf_R.obj; visual mesh filename=package://ares1_description/meshes/visual/calf_R.obj
- link right_thigh: geometry collision mesh filename=package://ares1_description/meshes/collision/thigh_R.obj; visual mesh filename=package://ares1_description/meshes/visual/thigh_R.obj
- link right_upper_arm: geometry collision mesh filename=package://ares1_description/meshes/collision/upper_arm_R.obj; visual mesh filename=package://ares1_description/meshes/visual/upper_arm_R.obj
- link sensor_dome: geometry 
- link shoulder_yoke: geometry 
Joints:
- removed joint drone1_fixed
- removed joint drone2_fixed
- removed joint left_rifle_joint
- removed joint pod_left_joint
- removed joint pod_right_joint
- removed joint right_launcher_joint
- removed joint shield_pivot
- joint abdomen1_fixed: origin xyz=0 0 0.115 rpy=0 0 0 -> xyz=0 0 0.274 rpy=0 0 0
- joint abdomen2_fixed: origin xyz=0 0 0.085 rpy=0 0 0 -> xyz=0 0 0.266 rpy=0 0 0
- joint abdomen3_fixed: origin xyz=0 0 0.085 rpy=0 0 0 -> xyz=0 0 0.266 rpy=0 0 0
- joint chest_joint: origin xyz=0 0 0.225 rpy=0 0 0 -> xyz=0 0 0.311 rpy=0 0 0
- joint head_joint: origin xyz=0 0 0.07 rpy=0 0 0 -> xyz=0 0 0.155 rpy=0 0 0
- joint neck_yaw: origin xyz=0 0 0.250 rpy=0 0 0 -> xyz=0 0 0.261 rpy=0 0 0
